File: data_collection/rover/rover_v3.1/power_board_v1/kicad/power_board_v1.kicad_sch (KiCad schematic)
At the start: 133 parts, among them J1 XT60_BATT, J10 from Pi USB2, J11 UPDI prog (UPDI/3V3/GND), J12 XT30 fallback pads, J13 USB_A port3 (3A), J14 from Pi USB3, J2 PANEL_SW, J3 USB4105-GF-A (TH shell), J4 USB_A radio1, J5 USB_A radio2, J6 AUX 5V 2A, J7 PI GPIO harness, J8 AUX_CTL out (JST-GH), J9 from Pi USB1, Q2 CSD18543Q3A diode, Q3 CSD18543Q3A switch, U1 LM5145 rail A, U10 TPS2557 ~3A (always on), U2 LM5145 rail B, U3 ATtiny816 (VQFN), U4 LM74800-Q1, U5 INA226 (addr 0x40), U6 TPS7A1633 3V3 60V LDO, U7 TPS2557 ~3A, U8 TPS2557 ~3A, U9 AP2112K-3.3 (switched)

Commit message: schematic v5: section boxes + validated structure links; U3 SOIC / J12 sync
Readability restructure of the generated schematic (netlist-neutral,
verified: netlist parity PASS vs previous sch modulo the U3 QFN->SOIC pin
map, 100 nets identical):
- 7 titled section boxes (input, front-end, supervisor, buck A, buck B,
  USB, harness) drawn from auto-tracked extents with title-clear padding.
- ~45 dashed guide polylines for the topology-carrying chains (battery
  path, FE b2b pair + EN/OV ladder, buck gate drives / SW node / LC /
  FB dividers / comp networks, USB port chains, sense dividers, I2C
  pulls). Links are GRAPHICS, never wires - link() asserts both endpoints
  already share a net, so a wrong link is a build error, and routing is
  side-aware so lines never cross symbol bodies.
- Regeneration syncs documentation with the board: U3 shown as SOIC-20
  with remapped pins, J12 as the DNP pigtail header. Title block rev v5.
- Fresh-eyes agent review drove 16 position fixes: stacked-cap banks to
  10mm pitch (refdes/value collisions), supervisor D5/U6 hotspot spread,
  J2/C17 moved inside the frame, C1/C2 clear of Q3 caption, short title
  block comments (were clipped off-sheet).
- Generator no longer overwrites power_board_v1.kicad_pro (it carries the
  v4.4 DRC-clean rule floors and severity policy).

Co-Authored-By: Claude Fable 5 <noreply@anthropic.com>
Parts:
- J12: value XT30 fallback pads -> 5V_A pigtail hdr DNP; footprint Connector_AMASS:AMASS_XT30PW-M_1x02_P2.50mm_Horizontal -> Connector_PinHeader_2.54mm:PinHeader_1x02_P2.54mm_Vertical
- U3: value ATtiny816 (VQFN) -> ATtiny816 (SOIC-20); footprint Package_DFN_QFN:QFN-20-1EP_3x3mm_P0.4mm_EP1.65x1.65mm -> Package_SO:SOIC-20W_7.5x12.8mm_P1.27mm
Connections:
- net AUX_CTL: now also U3.8 (PB3/AUX_CTL); no longer U3.11 (PB3/AUX_CTL)
- net EN_A: now also U3.6 (PB5/BUCKA_EN); no longer U3.9 (PB5/BUCKA_EN)
- net EN_USB1: now also U3.17 (PA1/USB_EN1); no longer U3.20 (PA1/USB_EN1)
- net EN_USB2: now also U3.18 (PA2/USB_EN2); no longer U3.1 (PA2/USB_EN2)
- net FAULT_USB: now also U3.3 (PA5/FAULT_USB); no longer U3.6 (PA5/FAULT_USB)
- net FE_EN: now also U3.7 (PB4/FE_EN); no longer U3.10 (PB4/FE_EN)
- net GND: now also U3.20 (GND); no longer U3.21 (EP), U3.3 (GND)
- net LED_STAT: now also U3.19 (PA3/LED); no longer U3.2 (PA3/LED)
- net LOW_BATT: now also U3.14 (PC2/LOW_BATT); no longer U3.17 (PC2/LOW_BATT)
- net MCU_3V3: now also U3.1 (VDD); no longer U3.4 (VDD)
- net NTC: now also U3.5 (PA7/NTC); no longer U3.8 (PA7/NTC)
- net PGOOD_A: now also U3.12 (PC0/PGOOD_A); no longer U3.15 (PC0/PGOOD_A)
- net PGOOD_B: now also U3.13 (PC1/PGOOD_B); no longer U3.16 (PC1/PGOOD_B)
- net SCL: now also U3.11 (PB0/SCL); no longer U3.14 (PB0/SCL)
- net SDA: now also U3.10 (PB1/SDA); no longer U3.13 (PB1/SDA)
- net SHDN_ACK: now also U3.15 (PC3/SHDN_ACK); no longer U3.18 (PC3/SHDN_ACK)
- net SW_SENSE: now also U3.9 (PB2/SW_SENSE); no longer U3.12 (PB2/SW_SENSE)
- net UPDI: now also U3.16 (PA0/UPDI); no longer U3.19 (PA0/UPDI)
- net V5A_SENSE: now also U3.4 (PA6/V5A_SENSE); no longer U3.7 (PA6/V5A_SENSE)
- net VSENSE: now also U3.2 (PA4/VIN_SENSE); no longer U3.5 (PA4/VIN_SENSE)

Commit message: power_board v4.5: add D8 (USB port 3 ESD array) — caught by KiCad 10 schematic-parity
KiCad 10.0.4 re-validation found D8 (USBLC6-2SC6, port 3 ESD) in the
schematic/netlist but absent from the board since v4: the 3-port change
added D8's place() call but not its REF_FP footprint entry, and
generate_board.py silently skipped footprint-less parts. Port 3 data
lines (J14->J13) carried no ESD protection while ports 1/2 had D2/D3.

- board: D8 placed at (138.25,74.16) south of J14; all 6 pads routed
  with exact-collide verification (data stubs F.Cu, VBUS3 via B.Cu lane,
  GND stub+via + pours); one redundant B.Cu GND stitch ripped (pour+plane
  carry GND; DRC 0 unconnected proves it). DRC: 0 violations, 0
  unconnected (severity-all, refill). Audit: PASS (same 3 known warns).
- generators: D8 added to REF_FP; missing footprint is now a HARD ERROR;
  netlist parser whitespace-tolerant (KiCad 10 pretty-prints netlists)
  with parsed-0 guards
- netlist.net regenerated (D8 complete + stale pre-SOIC U3 numbering)
- audit_board.py: KiCad >=9 compat (EDA_UNITS rename; WriteDRCReport
  segfaults headless -> kicad-cli drc fallback)
- fab/: full re-export on KiCad 10 (In1/In2 now .g1/.g2 - v10 protel
  naming; stale v7 gerbers + unused User_* layers removed), BOM line
  USBLC6-2SC6 now D2,D3,D8; upload zip added
- .kicad_pro: KiCad 10 format migration (float cleanup + new keys only;
  all rule floors and severities preserved, .kicad_dru untouched)
- .claude/settings.json: read-only tool allowlist (kicad-cli exports,
  pdftoppm/pdfinfo, rsvg-convert, nvidia-smi queries)
- docs/learnings.md: the silent-skip lesson + parity gate rule

Co-Authored-By: Claude Fable 5 <noreply@anthropic.com>
Parts:
- D8: footprint (none) -> Package_TO_SOT_SMD:SOT-23-6
