File: data_collection/rover/rover_v3.1/power_board_v1/kicad/power_board_v1.kicad_pcb (KiCad board)
At the start: 4 copper layers, 100 x 65 mm, 137 parts, among them J1 XT60_BATT, J10 from Pi USB2, J11 UPDI prog (UPDI/3V3/GND), J12 5V_A pigtail (DNP), J13 USB_A port3 (3A), J14 from Pi USB3, J2 PANEL_SW, J3 USB4105-GF-A (TH shell), J4 USB_A radio1, J5 USB_A radio2, J6 AUX 5V 2A, J7 PI GPIO harness, J8 AUX_CTL out (JST-GH), J9 from Pi USB1, Q2 CSD18543Q3A diode, Q3 CSD18543Q3A switch, U1 LM5145 rail A, U10 TPS2557 ~3A (always on), U2 LM5145 rail B, U3 ATtiny1616-SN (816-compat), U4 LM74800-Q1, U5 INA226 (addr 0x40), U6 TPS7A1633 3V3 60V LDO, U7 TPS2557 ~3A, U8 TPS2557 ~3A, U9 AP2112K-3.3 (switched)

Commit message: power_board v4.9: 6A switch-node copper was 0.15mm thin-pass tracks — added power pours
SW_A and SW_B (FET half-bridge -> inductor, ~6A + ripple) were routed
ONLY in 0.15mm KRT thin-pass tracks — a fuse, not a trace. Found by
manual current-path review; invisible to DRC/audit (no ampacity checks).

- F.Cu pour patches (priority 3): SW_A 83mm2, SW_B 57mm2 (compact switch
  nodes), 5V_A 126mm2 (LA1 -> caps/plane, +4 stitch vias), 5VB_PRE 171mm2
  (LB1 -> CB6x bank -> L4 pi-filter; net has no inner plane — the pour is
  the highway), 5V_B pad at L4 output (+3 plane vias)
- misrouted first attempt (5V_B patch on the 5VB_PRE section) ripped
- DRC 0 violations / 0 unconnected, audit PASS, fab + zip rebuilt
- docs/learnings.md: standing >1A copper-walk rule

Co-Authored-By: Claude Fable 5 <noreply@anthropic.com>
Routing:
- net 5V_B: vias 21 -> 24
- net 5V_A: vias 12 -> 16
- added copper zone on F.Cu, net 5VB_PRE
- added copper zone on F.Cu, net 5V_A
- added copper zone on F.Cu, net 5V_B
- added copper zone on F.Cu, net SW_A
- added copper zone on F.Cu, net SW_B
Changed lines of the file:
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@@
 	)
 	(via
+		(at 116.6 80)
+		(size 0.45)
+		(drill 0.2)
+		(layers "F.Cu" "B.Cu")
+		(net "5V_B")
+	)
+	(via
+		(at 116.23 81.03)
+		(size 0.45)
+		(drill 0.2)
+		(layers "F.Cu" "B.Cu")
+		(net "5V_B")
+	)
+	(via
 		(at 133.1 63)
 		(size 0.6)
@@
 	)
 	(via
+		(at 116.5 80.55)
+		(size 0.45)
+		(drill 0.2)
+		(layers "F.Cu" "B.Cu")
+		(net "5V_B")
+	)
+	(via
 		(at 87.5 104.8)
 		(size 0.6)
@@
 	)
 	(via
+		(at 112.2 59)
+		(size 0.45)
+		(drill 0.2)
+		(layers "F.Cu" "B.Cu")
+		(net "5V_A")
+	)
+	(via
 		(at 62 105.5)
 		(size 0.6)
@@
 	)
 	(via
+		(at 111.87 59.9)
+		(size 0.45)
+		(drill 0.2)
+		(layers "F.Cu" "B.Cu")
+		(net "5V_A")
+	)
+	(via
+		(at 112.12 59.48)
+		(size 0.45)
+		(drill 0.2)
+		(layers "F.Cu" "B.Cu")
+		(net "5V_A")
+	)
+	(via
 		(at 78.9 65.5)
 		(size 0.6)
@@
 		(net "5V_A")
 	)
+	(via
+		(at 111.5 60.21)
+		(size 0.45)
+		(drill 0.2)
+		(layers "F.Cu" "B.Cu")
+		(net "5V_A")
+	)
 	(segment
 		(start 60.7 106.9)
@@
 			)
 		)
+	)
+	(zone
+		(net "5V_B")
+		(layer "F.Cu")
+		(hatch edge 0.5)
+		(priority 3)
+		(connect_pads yes
+			(clearance 0.25)
+		)
+		(min_thickness 0.3)
+		(fill yes
+			(thermal_gap 0.5)
+			(thermal_bridge_width 0.5)
+			(island_removal_mode 0)
+		)
+		(polygon
+			(pts
+				(xy 113.8 77) (xy 122 77) (xy 122 83.5) (xy 113.8 83.5)
+			)
+		)
+	)
+	(zone
+		(net "SW_A")
+		(layer "F.Cu")
+		(hatch edge 0.5)
+		(priority 3)
+		(connect_pads yes
+			(clearance 0.25)
+		)
+		(min_thickness 0.3)
+		(fill yes
+			(thermal_gap 0.5)
+			(thermal_bridge_width 0.5)
+			(island_removal_mode 0)
+		)
+		(polygon
+			(pts
+				(xy 95.4 53.2) (xy 103.8 53.2) (xy 103.8 65.5) (xy 95.4 65.5)
+			)
+		)
+	)
+	(zone
+		(net "SW_B")
+		(layer "F.Cu")
+		(hatch edge 0.5)
+		(priority 3)
+		(connect_pads yes
+			(clearance 0.25)
+		)
+		(min_thickness 0.3)
+		(fill yes
+			(thermal_gap 0.5)
+			(thermal_bridge_width 0.5)
+			(island_removal_mode 0)
+		)
+		(polygon
+			(pts
+				(xy 95.4 85.2) (xy 103.8 85.2) (xy 103.8 97.5) (xy 95.4 97.5)
+			)
+		)
+	)
+	(zone
+		(net "5V_A")
+		(layer "F.Cu")
+		(hatch edge 0.5)
+		(priority 3)
+		(connect_pads yes
+			(clearance 0.25)
+		)
+		(min_thickness 0.3)
+		(fill yes
+			(thermal_gap 0.5)
+			(thermal_bridge_width 0.5)
+			(island_removal_mode 0)
+		)
+		(polygon
+			(pts
+				(xy 108.2 53) (xy 119.5 53) (xy 119.5 65.5) (xy 108.2 65.5)
+			)
+		)
+	)
+	(zone
+		(net "5VB_PRE")
+		(layer "F.Cu")
+		(hatch edge 0.5)
+		(priority 3)
+		(connect_pads yes
+			(clearance 0.25)
+		)
+		(min_thickness 0.3)
+		(fill yes
+			(thermal_gap 0.5)
+			(thermal_bridge_width 0.5)
+			(island_removal_mode 0)
+		)
+		(polygon
+			(pts
+				(xy 107.5 78.5) (xy 121 78.5) (xy 121 98.5) (xy 107.5 98.5)
+			)
+		)
